File: design_files/AST1015.brd (EAGLE design)
At the start: 10 x 10 mm, 4 parts, among them J1 SM05B, J2 SKTHBA

Commit message: updated documentation
Parts:
- removed J2: SKTHBA, tinycircuits:SKTHBA_TACT
- added SW1: PTS815, tinycircuits:PTS815
- J1: device tinycircuits:JST_SH_5X1 -> tinycircuits:JST_SH_5X1_EDGE
Connections:
- net GND: now also SW1.1, SW1.2; no longer J2.1, J2.2
- net INT: now also SW1.3, SW1.4; no longer J2.3, J2.4
Other:
- board text added: "Small"
- board text added: "Wireling Small Button"
- board text removed: "Momentary"
- board text removed: "Momentary Pushbutton Board"
Changed lines of the file:
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@@
 <layer number="54" name="bGND_GNDA" color="7" fill="1" visible="yes" active="yes"/>
 <layer number="56" name="wert" color="7" fill="1" visible="yes" active="yes"/>
+<layer number="57" name="tCAD" color="7" fill="1" visible="no" active="no"/>
+<layer number="58" name="bCAD" color="7" fill="1" visible="no" active="no"/>
+<layer number="59" name="Invisible" color="7" fill="1" visible="no" active="no"/>
+<layer number="61" name="stand" color="7" fill="1" visible="no" active="no"/>
+<layer number="88" name="SimResults" color="9" fill="1" visible="yes" active="yes"/>
+<layer number="89" name="SimProbes" color="9" fill="1" visible="yes" active="yes"/>
+<layer number="90" name="Modules" color="5" fill="1" visible="yes" active="yes"/>
 <layer number="91" name="Nets" color="2" fill="1" visible="no" active="no"/>
 <layer number="92" name="Busses" color="1" fill="1" visible="no" active="no"/>
@@
 <layer number="97" name="Info" color="7" fill="1" visible="no" active="no"/>
 <layer number="98" name="Guide" color="6" fill="1" visible="no" active="no"/>
+<layer number="99" name="SpiceOrder" color="5" fill="1" visible="no" active="no"/>
 <layer number="100" name="Muster" color="7" fill="1" visible="yes" active="yes"/>
 <layer number="101" name="Patch_Top" color="7" fill="1" visible="yes" active="yes"/>
@@
 <layer number="111" name="tGTest" color="4" fill="1" visible="no" active="no"/>
 <layer number="112" name="bGTest" color="1" fill="1" visible="no" active="no"/>
+<layer number="113" name="HENWAY_PKG" color="12" fill="1" visible="yes" active="yes"/>
+<layer number="114" name="50_Electronics_Plate" color="7" fill="1" visible="yes" active="yes"/>
+<layer number="115" name="henwayRES" color="5" fill="1" visible="yes" active="yes"/>
 <layer number="116" name="Patch_BOT" color="7" fill="1" visible="yes" active="yes"/>
 <layer number="117" name="mPads" color="7" fill="1" visible="no" active="no"/>
@@
 <layer number="151" name="HeatSink" color="7" fill="1" visible="yes" active="yes"/>
 <layer number="152" name="mbDocu" color="7" fill="1" visible="no" active="no"/>
+<layer number="153" name="FabDoc1" color="6" fill="1" visible="no" active="no"/>
+<layer number="154" name="FabDoc2" color="2" fill="1" visible="no" active="no"/>
+<layer number="155" name="FabDoc3" color="7" fill="15" visible="no" active="no"/>
+<layer number="156" name="bCapacitor" color="7" fill="1" visible="yes" active="yes"/>
+<layer number="157" name="tResistor" color="7" fill="1" visible="yes" active="yes"/>
+<layer number="158" name="bResistor" color="7" fill="1" visible="yes" active="yes"/>
+<layer number="159" name="henwayCAP" color="13" fill="1" visible="yes" active="yes"/>
+<layer number="160" name="IDFDebug" color="7" fill="1" visible="yes" active="yes"/>
 <layer number="191" name="mNets" color="7" fill="1" visible="no" active="no"/>
 <layer number="192" name="mBusses" color="7" fill="1" visible="no" active="no"/>
@@
 <layer number="223" name="223bmp" color="7" fill="1" visible="yes" active="yes"/>
 <layer number="224" name="224bmp" color="7" fill="1" visible="yes" active="yes"/>
+<layer number="231" name="Eagle3D_PG1" color="7" fill="1" visible="yes" active="yes"/>
+<layer number="232" name="Eagle3D_PG2" color="7" fill="1" visible="yes" active="yes"/>
+<layer number="233" name="Eagle3D_PG3" color="7" fill="1" visible="yes" active="yes"/>
 <layer number="248" name="Housing" color="7" fill="1" visible="yes" active="yes"/>
 <layer number="249" name="Edge" color="7" fill="1" visible="yes" active="yes"/>
@@
 <wire x1="0" y1="40.8" x2="0" y2="0" width="0.127" layer="48"/>
 <dimension x1="15" y1="20" x2="25" y2="20" x3="20" y3="21.454653125" layer="48"/>
-<text x="38.111025" y="4.365003125" size="0.889" layer="48">Momentary Pushbutton Board</text>
+<text x="38.111025" y="4.365003125" size="0.889" layer="48">Wireling Small Button</text>
 <text x="34.986825" y="1.7714" size="0.889" layer="48">AS-PCB-AST1015</text>
 <text x="57.3810375" y="1.6952" size="0.889" layer="48">1</text>
@@
 <rectangle x1="18.747940625" y1="13.71801875" x2="19.027340625" y2="13.72309375" layer="22"/>
 <rectangle x1="20.8155" y1="13.71801875" x2="21.08981875" y2="13.72309375" layer="22"/>
-<text x="21.5" y="16.4" size="0.76" layer="22" rot="SMR0">Momentary</text>
+<text x="21.5" y="16.4" size="0.76" layer="22" rot="SMR0">Small</text>
 <wire x1="22" y1="14.45" x2="23.15" y2="15.65" width="0.1" layer="22"/>
 <wire x1="22" y1="15.05" x2="22.55" y2="15.6" width="0.1" layer="22"/>
@@
 <attribute name="NO_BOM" value="TRUE" x="34" y="0" size="1.778" layer="27" display="off"/>
 </element>
-<element name="J1" library="tinycircuits" package="JST_SH_5X1" value="SM05B" x="20" y="12.125">
+<element name="J1" library="tinycircuits" package="JST_SH_5X1_EDGE" value="SM05B" x="20" y="12.125">
 <attribute name="PARTNO" value="AS-ITM-00340" x="20" y="12.125" size="1.778" layer="27" display="off"/>
 <attribute name="VALUE" value="SM05B" x="20" y="12.125" size="1.778" layer="27" display="off"/>
@@
 <attribute name="VALUE" value="10.0K" x="24.1" y="13.9" size="1.778" layer="27" rot="R270" display="off"/>
 </element>
-<element name="J2" library="tinycircuits" package="SKTHBA_TACT" value="SKTHBA" x="20" y="17.1" rot="R180">
-<attribute name="PARTNO" value="AS-ITM-00369" x="20" y="17.1" size="1.778" layer="27" rot="R180" display="off"/>
-<attribute name="VALUE" value="SKTHBA" x="20" y="17.1" size="1.778" layer="27" rot="R180" display="off"/>
+<element name="SW1" library="tinycircuits" package="PTS815" value="PTS815" x="20" y="17.2">
+<attribute name="PARTNO" value="AS-ITM-00544" x="20" y="17.2" size="1.778" layer="27" display="off"/>
+<attribute name="VALUE" value="PTS815" x="20" y="17.2" size="1.778" layer="27" display="off"/>
 </element>
 </elements>
@@
 <via x="18.3" y="19.2" extent="1-16" drill="0.381"/>
 <via x="21.7" y="19.2" extent="1-16" drill="0.381"/>
-<contactref element="J2" pad="1"/>
-<contactref element="J2" pad="2"/>
+<contactref element="SW1" pad="1"/>
+<contactref element="SW1" pad="2"/>
 </signal>
 <signal name="N$13">
@@
 <contactref element="J1" pad="5"/>
 <contactref element="R1" pad="1"/>
-<contactref element="J2" pad="3"/>
-<contactref element="J2" pad="4"/>
-<wire x1="18.025" y1="16.45" x2="21.975" y2="16.45" width="0.4064" layer="1"/>
 <wire x1="22" y1="14.6" x2="21.975" y2="14.6" width="0.4064" layer="1"/>
-<wire x1="21.975" y1="14.6" x2="21.975" y2="16.45" width="0.4064" layer="1"/>
 <wire x1="24.1" y1="14.5" x2="22" y2="14.5" width="0.4064" layer="1"/>
 <wire x1="22" y1="14.5" x2="22" y2="14.6" width="0.4064" layer="1"/>
+<contactref element="SW1" pad="3"/>
+<contactref element="SW1" pad="4"/>
+<wire x1="22" y1="14.6" x2="22" y2="16.1" width="0.2032" layer="1"/>
+<wire x1="22" y1="16.1" x2="18" y2="16.1" width="0.2032" layer="1"/>
 </signal>
 </signals>
