File: design_files/AST1015.sch (EAGLE design)
At the start: 3 parts, among them J1 SM05B, J2 SKTHBA

Commit message: updated documentation
Parts:
- removed J2: SKTHBA, tinycircuits:AS-ITM-00369
- added SW1: PTS815, tinycircuits:AS-ITM-00544
- J1: device tinycircuits:AS-ITM-00340 -> tinycircuits:AS-ITM-00340EDGE
Connections:
- net GND: now also SW1.1, SW1.3; no longer J2.1, J2.2
- net INT: now also SW1.2, SW1.4; no longer J2.3, J2.4
Other:
- note added: "Hand Populated: -"
- note added: "Hand Soldered: -"
- note added: "Non Populated: -"
- note added: "Notes: -"
- note added: "Variant: Standard - R"
- note added: "Wireling Small Button"
- note removed: "Momentary Pushbutton Board"
- note removed: "NOTES:"
